Commit message: ros2 control working, next work on teleop

File: description/prac_robot.urdf.xacro (robot description, xacro)
@@ -1,6 +1,155 @@
 <?xml version="1.0"?>
 <robot xmlns:xacro="http://www.ros.org/wiki/xacro"  name="robot">
-    <xacro:arg name="use_ros2_control" default="true"/>
-    <xacro:arg name="sim_mode" default="false"/>
-    <xacro:include filename="prac_robot_core.xacro" />
+    <!-- This will include all the contents of example_include.xacro first. Go check it out! -->
+    <xacro:include filename="prac_include.xacro" />
+    <xacro:include filename="ros2_control.xacro" />
+    <!-- my own stuff -->
+    <xacro:include filename="inertial_macros.xacro"/>
+    <xacro:property name="chassis_length" value="1"/>
+    <xacro:property name="chassis_width" value="0.6"/>
+    <xacro:property name="chassis_height" value="0.4"/>
+    <xacro:property name="chassis_mass" value="1.0"/>
+    <xacro:property name="wheel_radius" value="0.2"/>
+    <xacro:property name="wheel_thickness" value="0.1"/>
+    <xacro:property name="wheel_mass" value="0.1"/>
+    <xacro:property name="wheel_offset_x" value="0.5"/>
+    <xacro:property name="wheel_offset_y" value="0.35"/>
+    <xacro:property name="wheel_offset_z" value="-0.2"/>
+    <xacro:property name="caster_wheel_radius" value="0.05"/>
+    <xacro:property name="caster_wheel_mass" value="0.01"/>
+    <xacro:property name="caster_wheel_offset_x" value="0.4"/>
+    <xacro:property name="caster_wheel_offset_z" value="${wheel_offset_z - wheel_radius + caster_wheel_radius}"/>
+    <!-- my own stuff -->
+    <!-- xacro need this dummy -->
+    <link name="dummy"></link>
+    <!-- A simple fixed joint from our empty a link, to our base. -->
+    <!-- The base origin is offset from the a origin. -->
+    <joint name="dummy_joint" type="fixed">
+        <parent link="dummy"/>
+        <child link="chassis"/>
+    </joint>
+    <!-- chassis is a large rectangular plate. Some things to note: -->
+    <!-- - We set the visual origin Z to half the box height, so that the link origin sits at the bottom of the box -->
+    <!-- - We set the collision to be identical to the visual -->
+    <!-- - We specified the colour manually (but still need to enter a name) -->
+    <!-- - We specified all the inertial parameters manually -->
+    <link name="chassis">
+        <visual>
+            <origin xyz="0 0 0" rpy="0 0 0"/>
+            <geometry>
+                <box size="${chassis_length} ${chassis_width} ${chassis_height}" />
+            </geometry>
+            <material name="green">
+                <color rgba="0.2 1 0.2 1"/>
+            </material>
+        </visual>
+        <collision>
+            <origin xyz="0 0 0" rpy="0 0 0"/>
+            <geometry>
+                <box size="${chassis_length} ${chassis_width} ${chassis_height}" />
+            </geometry>
+        </collision>
+        <xacro:inertial_box mass="10" x="${chassis_length}" y="${chassis_length}" z="${chassis_length}">
+            <origin xyz="0 0 0" rpy="0 0 0"/>
+        </xacro:inertial_box>
+    </link>
+    <!-- LEFT WHEEL -->
+    <joint name="left_wheel_joint" type="continuous">
+        <parent link="chassis"/>
+        <child link="left_wheel"/>
+        <origin xyz="0 ${wheel_offset_y} ${wheel_offset_z}" rpy="-${pi/2} 0 0" />
+        <axis xyz="0 0 1"/>
+    </joint>
+    <link name="left_wheel">
+        <visual>
+            <geometry>
+                <cylinder radius="${wheel_radius}" length="${wheel_thickness}"/>
+            </geometry>
+            <material name="blue">
+                <color rgba="0 0 0.075"/>
+            </material>
+        </visual>
+        <collision>
+            <geometry>
+                <sphere radius="${wheel_radius}"/>
+            </geometry>
+        </collision>
+        <xacro:inertial_cylinder mass="${wheel_mass}" length="${wheel_thickness}" radius="${wheel_radius}">
+            <origin xyz="0 0 0" rpy="0 0 0"/>
+        </xacro:inertial_cylinder>
+    </link>
+    <!-- Right WHEEL -->
+    <joint name="right_wheel_joint" type="continuous">
+        <parent link="chassis"/>
+        <child link="right_wheel"/>
+        <origin xyz="0 ${-wheel_offset_y} ${wheel_offset_z}" rpy="${pi/2} 0 0" />
+        <axis xyz="0 0 -1"/>
+    </joint>
+    <link name="right_wheel">
+        <visual>
+            <geometry>
+                <cylinder radius="${wheel_radius}" length="${wheel_thickness}"/>
+            </geometry>
+            <material name="blue">
+                <color rgba="0 0 0.075"/>
+            </material>
+        </visual>
+        <collision>
+            <geometry>
+                <sphere radius="${wheel_radius}"/>
+            </geometry>
+        </collision>
+        <xacro:inertial_cylinder mass="${wheel_mass}" length="${wheel_thickness}" radius="${wheel_radius}">
+            <origin xyz="0 0 0" rpy="0 0 0"/>
+        </xacro:inertial_cylinder>
+    </link>
+    <!-- front Castor wheel-->
+    <joint name="front_caster_wheel_joint" type="fixed">
+        <parent link="chassis"/>
+        <child link="front_caster_wheel"/>
+        <origin xyz="${caster_wheel_offset_x} 0 ${caster_wheel_offset_z}"/>
+    </joint>
+    <link name="front_caster_wheel">
+        <visual>
+            <geometry>
+                <sphere radius="${caster_wheel_radius}"/>
+            </geometry>
+            <material name="blue">
+                <color rgba="0 0 0.075"/>
+            </material>
+        </visual>
+        <collision>
+            <geometry>
+                <sphere radius="${caster_wheel_radius}"/>
+            </geometry>
+        </collision>
+        <xacro:inertial_sphere mass="${caster_wheel_mass}" radius="${caster_wheel_radius}">
+            <origin xyz="0 0 0" rpy="0 0 0"/>
+        </xacro:inertial_sphere>
+    </link>
+    <!-- rear Castor wheel-->
+    <joint name="rear_caster_wheel_joint" type="fixed">
+        <parent link="chassis"/>
+        <child link="rear_caster_wheel"/>
+        <origin xyz="${-caster_wheel_offset_x} 0 ${caster_wheel_offset_z}"/>
+    </joint>
+    <link name="rear_caster_wheel">
+        <visual>
+            <geometry>
+                <sphere radius="${caster_wheel_radius}"/>
+            </geometry>
+            <material name="blue">
+                <color rgba="0 0 0.075"/>
+            </material>
+        </visual>
+        <collision>
+            <geometry>
+                <sphere radius="${caster_wheel_radius}"/>
+            </geometry>
+        </collision>
+        <xacro:inertial_sphere mass="${caster_wheel_mass}" radius="${caster_wheel_radius}">
+            <origin xyz="0 0 0" rpy="0 0 0"/>
+        </xacro:inertial_sphere>
+    </link>
+    <xacro:include filename="example_gazebo.xacro" />
 </robot>

File: description/ros2_control.xacro (robot description, xacro)
@@ -1,62 +1,30 @@
 <?xml version="1.0"?>
 <robot xmlns:xacro="http://www.ros.org/wiki/xacro">
-    <xacro:unless value="$(arg sim_mode)">
-        <ros2_control name="RealRobot" type="system">
-            <hardware>
-                <plugin>diffdrive_arduino/DiffDriveArduinoHardware</plugin>
-                <param name="left_wheel_name">left_wheel_joint</param>
-                <param name="right_wheel_name">right_wheel_joint</param>
-                <param name="loop_rate">30</param>
-                <param name="device">/dev/ttyUSB0</param>
-                <param name="baud_rate">57600</param>
-                <param name="timeout_ms">1000</param>
-                <param name="enc_counts_per_rev">3436</param>
-            </hardware>
-            <joint name="left_wheel_joint">
-                <command_interface name="velocity">
-                    <param name="min">-10</param>
-                    <param name="max">10</param>
-                </command_interface>
-                <state_interface name="position"/>
-                <state_interface name="velocity"/>
-            </joint>
-            <joint name="right_wheel_joint">
-                <command_interface name="velocity">
-                    <param name="min">-10</param>
-                    <param name="max">10</param>
-                </command_interface>
-                <state_interface name="position"/>
-                <state_interface name="velocity"/>
-            </joint>
-        </ros2_control>
-    </xacro:unless>
-    <xacro:if value="$(arg sim_mode)">
-        <ros2_control name="GazeboSystem" type="system">
-            <hardware>
-                <plugin>gazebo_ros2_control/GazeboSystem</plugin>
-            </hardware>
-            <joint name="left_wheel_joint">
-                <command_interface name="velocity">
-                    <param name="min">-10</param>
-                    <param name="max">10</param>
-                </command_interface>
-                <state_interface name="velocity"/>
-                <state_interface name="position"/>
-            </joint>
-            <joint name="right_wheel_joint">
-                <command_interface name="velocity">
-                    <param name="min">-10</param>
-                    <param name="max">10</param>
-                </command_interface>
-                <state_interface name="velocity"/>
-                <state_interface name="position"/>
-            </joint>
-        </ros2_control>
-    </xacro:if>
-    <gazebo>
-        <plugin name="gazebo_ros2_control" filename="libgazebo_ros2_control.so">
-            <parameters>$(find prac_robot)/config/my_controllers.yaml</parameters>
-            <parameters>$(find prac_robot)/config/gaz_ros2_ctl_use_sim.yaml</parameters>
-        </plugin>
-    </gazebo>
+  <ros2_control name="IgnitionSystem" type="system">
+    <hardware>
+      <plugin>ign_ros2_control/IgnitionSystem</plugin>
+    </hardware>
+    <joint name="left_wheel_joint">
+      <command_interface name="velocity">
+        <param name="min">-1</param>
+        <param name="max">1</param>
+      </command_interface>
+      <state_interface name="position"/>
+      <state_interface name="velocity"/>
+    </joint>
+    <joint name="right_wheel_joint">
+      <command_interface name="velocity">
+        <param name="min">-1</param>
+        <param name="max">1</param>
+      </command_interface>
+      <state_interface name="position"/>
+      <state_interface name="velocity"/>
+    </joint>
+  </ros2_control>
+  <gazebo>
+    <!-- Joint state publisher -->
+    <plugin filename="ign_ros2_control-system" name="ign_ros2_control::IgnitionROS2ControlPlugin">
+      <parameters>$(find prac_robot)/config/prac_controller.yaml</parameters>
+    </plugin>
+  </gazebo>
 </robot>

Commit message: trying to get lidar working

File: description/prac_robot.urdf.xacro (robot description, xacro)
@@ -4,4 +4,5 @@
     <xacro:include filename="prac_include.xacro" />
     <xacro:include filename="ros2_control.xacro" />
+    <xacro:include filename="lidar.xacro" />
     <!-- my own stuff -->
     <xacro:include filename="inertial_macros.xacro"/>
@@ -23,4 +24,10 @@
     <!-- xacro need this dummy -->
     <link name="dummy"></link>
+    <joint name="dummy_footprint_joint" type="fixed">
+        <parent link="dummy"/>
+        <child link="footprint"/>
+        <origin xyz="0 0 0" rpy="0 0 0"/>
+    </joint>
+    <link name= "footprint"></link>
     <!-- A simple fixed joint from our empty a link, to our base. -->
     <!-- The base origin is offset from the a origin. -->
@@ -28,4 +35,5 @@
         <parent link="dummy"/>
         <child link="chassis"/>
+        <origin xyz="${-wheel_offset_x} 0 ${-wheel_offset_z}"/>
     </joint>
     <!-- chassis is a large rectangular plate. Some things to note: -->

Commit message: fixed urdf and tf, need work on lidar, issue might be gazebo tf of lidar

File: description/prac_robot.urdf.xacro (robot description, xacro)
@@ -22,8 +22,8 @@
     <xacro:property name="caster_wheel_offset_z" value="${wheel_offset_z - wheel_radius + caster_wheel_radius}"/>
     <!-- my own stuff -->
-    <!-- xacro need this dummy -->
-    <link name="dummy"></link>
-    <joint name="dummy_footprint_joint" type="fixed">
-        <parent link="dummy"/>
+    <!-- xacro need this base_link -->
+    <link name="base_link"></link>
+    <joint name="base_footprint_joint" type="fixed">
+        <parent link="base_link"/>
         <child link="footprint"/>
         <origin xyz="0 0 0" rpy="0 0 0"/>
@@ -32,6 +32,6 @@
     <!-- A simple fixed joint from our empty a link, to our base. -->
     <!-- The base origin is offset from the a origin. -->
-    <joint name="dummy_joint" type="fixed">
-        <parent link="dummy"/>
+    <joint name="chassis_joint" type="fixed">
+        <parent link="base_link"/>
         <child link="chassis"/>
         <origin xyz="${-wheel_offset_x} 0 ${-wheel_offset_z}"/>
@@ -64,5 +64,5 @@
     <!-- LEFT WHEEL -->
     <joint name="left_wheel_joint" type="continuous">
-        <parent link="chassis"/>
+        <parent link="base_link"/>
         <child link="left_wheel"/>
         <origin xyz="0 ${wheel_offset_y} ${wheel_offset_z}" rpy="-${pi/2} 0 0" />
@@ -89,5 +89,5 @@
     <!-- Right WHEEL -->
     <joint name="right_wheel_joint" type="continuous">
-        <parent link="chassis"/>
+        <parent link="base_link"/>
         <child link="right_wheel"/>
         <origin xyz="0 ${-wheel_offset_y} ${wheel_offset_z}" rpy="${pi/2} 0 0" />

Commit message: fixed urdf again

File: description/prac_robot.urdf.xacro (robot description, xacro)
@@ -14,7 +14,7 @@
     <xacro:property name="wheel_thickness" value="0.1"/>
     <xacro:property name="wheel_mass" value="0.1"/>
-    <xacro:property name="wheel_offset_x" value="0.5"/>
+    <xacro:property name="wheel_offset_x" value="0.2"/>
     <xacro:property name="wheel_offset_y" value="0.35"/>
-    <xacro:property name="wheel_offset_z" value="-0.2"/>
+    <xacro:property name="wheel_offset_z" value="-0.1"/>
     <xacro:property name="caster_wheel_radius" value="0.05"/>
     <xacro:property name="caster_wheel_mass" value="0.01"/>
@@ -66,5 +66,5 @@
         <parent link="base_link"/>
         <child link="left_wheel"/>
-        <origin xyz="0 ${wheel_offset_y} ${wheel_offset_z}" rpy="-${pi/2} 0 0" />
+        <origin xyz="0 ${wheel_offset_y} 0" rpy="-${pi/2} 0 0" />
         <axis xyz="0 0 1"/>
     </joint>
@@ -91,5 +91,5 @@
         <parent link="base_link"/>
         <child link="right_wheel"/>
-        <origin xyz="0 ${-wheel_offset_y} ${wheel_offset_z}" rpy="${pi/2} 0 0" />
+        <origin xyz="0 ${-wheel_offset_y} 0" rpy="${pi/2} 0 0" />
         <axis xyz="0 0 -1"/>
     </joint>
@@ -111,28 +111,4 @@
             <origin xyz="0 0 0" rpy="0 0 0"/>
         </xacro:inertial_cylinder>
-    </link>
-    <!-- front Castor wheel-->
-    <joint name="front_caster_wheel_joint" type="fixed">
-        <parent link="chassis"/>
-        <child link="front_caster_wheel"/>
-        <origin xyz="${caster_wheel_offset_x} 0 ${caster_wheel_offset_z}"/>
-    </joint>
-    <link name="front_caster_wheel">
-        <visual>
-            <geometry>
-                <sphere radius="${caster_wheel_radius}"/>
-            </geometry>
-            <material name="blue">
-                <color rgba="0 0 0.075"/>
-            </material>
-        </visual>
-        <collision>
-            <geometry>
-                <sphere radius="${caster_wheel_radius}"/>
-            </geometry>
-        </collision>
-        <xacro:inertial_sphere mass="${caster_wheel_mass}" radius="${caster_wheel_radius}">
-            <origin xyz="0 0 0" rpy="0 0 0"/>
-        </xacro:inertial_sphere>
     </link>
     <!-- rear Castor wheel-->
