Commit message: need to fix map and odom

File: prac_robot/description/lidar.xacro (robot description, xacro)
@@ -4,5 +4,5 @@
         <parent link="chassis"/>
         <child link="laser_frame"/>
-        <origin xyz="0.122 0 0.212" rpy="0 0 0"/>
+        <origin xyz="0.0 0 0.2" rpy="0 0 0"/>
     </joint>
     <link name="laser_frame">

File: prac_robot/description/prac_robot.urdf.xacro (robot description, xacro)
@@ -8,12 +8,12 @@
     <xacro:include filename="inertial_macros.xacro"/>
     <xacro:property name="chassis_length" value="1"/>
-    <xacro:property name="chassis_width" value="0.6"/>
+    <xacro:property name="chassis_width" value="0.7"/>
     <xacro:property name="chassis_height" value="0.4"/>
     <xacro:property name="chassis_mass" value="1.0"/>
-    <xacro:property name="wheel_radius" value="0.2"/>
+    <xacro:property name="wheel_radius" value="0.3"/>
     <xacro:property name="wheel_thickness" value="0.1"/>
     <xacro:property name="wheel_mass" value="0.1"/>
-    <xacro:property name="wheel_offset_x" value="0.2"/>
-    <xacro:property name="wheel_offset_y" value="0.35"/>
+    <xacro:property name="wheel_offset_x" value="0.0"/>
+    <xacro:property name="wheel_offset_y" value="0.4"/>
     <xacro:property name="wheel_offset_z" value="-0.1"/>
     <xacro:property name="caster_wheel_radius" value="0.05"/>
@@ -136,3 +136,27 @@
         </xacro:inertial_sphere>
     </link>
+    <!-- front Castor wheel-->
+    <joint name="front_caster_wheel_joint" type="fixed">
+        <parent link="chassis"/>
+        <child link="front_caster_wheel"/>
+        <origin xyz="${caster_wheel_offset_x} 0 ${caster_wheel_offset_z}"/>
+    </joint>
+    <link name="front_caster_wheel">
+        <visual>
+            <geometry>
+                <sphere radius="${caster_wheel_radius}"/>
+            </geometry>
+            <material name="blue">
+                <color rgba="0 0 0.075"/>
+            </material>
+        </visual>
+        <collision>
+            <geometry>
+                <sphere radius="${caster_wheel_radius}"/>
+            </geometry>
+        </collision>
+        <xacro:inertial_sphere mass="${caster_wheel_mass}" radius="${caster_wheel_radius}">
+            <origin xyz="0 0 0" rpy="0 0 0"/>
+        </xacro:inertial_sphere>
+    </link>
 </robot>
