Commit message: added ros2 control manager, need to refine car model and map slowly, maybe map bit by bit

File: prac_robot/description/prac_robot.urdf.xacro (robot description, xacro)
@@ -74,6 +74,6 @@
                 <cylinder radius="${wheel_radius}" length="${wheel_thickness}"/>
             </geometry>
-            <material name="blue">
-                <color rgba="0 0 0.075"/>
+            <material name="green">
+                <color rgba="0.2 1 0.2 1"/>
             </material>
         </visual>

Commit message: added map: depot_map

File: prac_robot/description/prac_robot.urdf.xacro (robot description, xacro)
@@ -7,17 +7,17 @@
     <!-- my own stuff -->
     <xacro:include filename="inertial_macros.xacro"/>
-    <xacro:property name="chassis_length" value="1"/>
-    <xacro:property name="chassis_width" value="0.7"/>
+    <xacro:property name="chassis_length" value="0.6"/>
+    <xacro:property name="chassis_width" value="0.4"/>
     <xacro:property name="chassis_height" value="0.4"/>
     <xacro:property name="chassis_mass" value="1.0"/>
-    <xacro:property name="wheel_radius" value="0.3"/>
+    <xacro:property name="wheel_radius" value="0.2"/>
     <xacro:property name="wheel_thickness" value="0.1"/>
     <xacro:property name="wheel_mass" value="0.1"/>
     <xacro:property name="wheel_offset_x" value="0.0"/>
-    <xacro:property name="wheel_offset_y" value="0.4"/>
+    <xacro:property name="wheel_offset_y" value="0.25"/>
     <xacro:property name="wheel_offset_z" value="-0.1"/>
     <xacro:property name="caster_wheel_radius" value="0.05"/>
     <xacro:property name="caster_wheel_mass" value="0.01"/>
-    <xacro:property name="caster_wheel_offset_x" value="0.4"/>
+    <xacro:property name="caster_wheel_offset_x" value="0.25"/>
     <xacro:property name="caster_wheel_offset_z" value="${wheel_offset_z - wheel_radius + caster_wheel_radius}"/>
     <!-- my own stuff -->

Commit message: modified README, A* is doggy need to fix, then start working on RRT*

File: prac_robot/description/prac_robot.urdf.xacro (robot description, xacro)
@@ -10,5 +10,5 @@
     <xacro:property name="chassis_width" value="0.4"/>
     <xacro:property name="chassis_height" value="0.4"/>
-    <xacro:property name="chassis_mass" value="1.0"/>
+    <xacro:property name="chassis_mass" value="0.5"/>
     <xacro:property name="wheel_radius" value="0.2"/>
     <xacro:property name="wheel_thickness" value="0.1"/>
